File: KeyboardTransformer.brd (EAGLE design)
At the start: 100 x 20 mm, 45 parts, among them IC1 74LS09N, IC2 ли6, IC6 74LS09N, IC7 74AC10N

Commit message: .
Parts:
- moved RV1 70.7 mm to (-42.5, 46.4), flipped to the bottom, turned to 180 degrees
Routing:
- net N$1: track 0.00 -> 20.5 mm
Changed lines of the file:
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@@
 <setting verticaltext="up"/>
 </settings>
-<grid distance="1" unitdist="mm" unit="mm" style="lines" multiple="1" display="yes" altdistance="0.025" altunitdist="inch" altunit="inch"/>
+<grid distance="25" unitdist="mil" unit="mil" style="lines" multiple="1" display="yes" altdistance="0.025" altunitdist="inch" altunit="inch"/>
 <layers>
 <layer number="1" name="Top" color="4" fill="1" visible="yes" active="yes"/>
@@
 <element name="R2A" library="rcl" package="M0805" value="11k" x="-25.4" y="110.49" rot="R90"/>
 <element name="C3" library="rcl" package="C0805" value="220p" x="-19.05" y="110.49" rot="R90"/>
-<element name="RV1" library="rcl" package="M0805" value="1k" x="-12.7" y="110.49" rot="R90"/>
+<element name="RV1" library="rcl" package="M0805" value="1k" x="-42.545" y="46.355" rot="MR180"/>
 <element name="DD4" library="74xx-eu" package="DIL14" value="К555ЛА9" x="-3.175" y="55.245"/>
 <element name="R7" library="rcl" package="M0805" value="1k" x="5.715" y="110.49" rot="R90"/>
@@
 <wire x1="-45.72" y1="17.2466" x2="-36.83" y2="5.08" width="0" layer="19" extent="1-16"/>
 <wire x1="-46.99" y1="31.115" x2="-45.72" y2="17.2466" width="0" layer="19" extent="16-16"/>
-<wire x1="-19.685" y1="27.305" x2="-45.72" y2="17.2466" width="0" layer="19" extent="16-16"/>
+<wire x1="-19.685" y1="27.305" x2="-46.99" y2="31.115" width="0" layer="19" extent="1-1"/>
 <wire x1="-15.875" y1="29.21" x2="-19.685" y2="27.305" width="0" layer="19" extent="1-1"/>
 <wire x1="-1.905" y1="30.48" x2="-14.605" y2="27.94" width="0" layer="19" extent="1-16"/>
 <wire x1="3.175" y1="31.115" x2="-0.635" y2="29.21" width="0" layer="19" extent="16-16"/>
 <wire x1="16.51" y1="31.115" x2="3.175" y2="31.115" width="0" layer="19" extent="1-1"/>
+<wire x1="30.48" y1="33.02" x2="16.51" y2="31.115" width="0" layer="19" extent="1-1"/>
 <wire x1="4.445" y1="51.435" x2="-14.605" y2="46.99" width="0" layer="19" extent="1-1"/>
-<wire x1="30.48" y1="33.02" x2="16.51" y2="31.115" width="0" layer="19" extent="1-1"/>
 <wire x1="36.83" y1="12.065" x2="30.48" y2="33.02" width="0" layer="19" extent="1-1"/>
 <wire x1="-27.305" y1="70.545" x2="-14.605" y2="46.99" width="0" layer="19" extent="1-1"/>
@@
 <wire x1="19.05" y1="121.6" x2="25.4" y2="121.6" width="0" layer="19" extent="1-1"/>
 <wire x1="5.715" y1="111.44" x2="19.05" y2="121.6" width="0" layer="19" extent="1-1"/>
-<wire x1="-12.7" y1="111.44" x2="5.715" y2="111.44" width="0" layer="19" extent="1-1"/>
-<wire x1="-25.4" y1="111.44" x2="-12.7" y2="111.44" width="0" layer="19" extent="1-1"/>
+<wire x1="-25.4" y1="111.44" x2="5.715" y2="111.44" width="0" layer="19" extent="1-1"/>
 <wire x1="-31.75" y1="111.44" x2="-25.4" y2="111.44" width="0" layer="19" extent="1-1"/>
 <wire x1="-29.21" y1="121.6" x2="-31.75" y2="111.44" width="0" layer="19" extent="1-1"/>
@@
 <wire x1="-27.305" y1="65.345" x2="-20.32" y2="66.99" width="0" layer="19" extent="1-1"/>
 <wire x1="-10.795" y1="59.055" x2="-20.32" y2="66.99" width="0" layer="19" extent="1-1"/>
-<wire x1="-34.925" y1="46.99" x2="-27.305" y2="65.345" width="0" layer="19" extent="1-1"/>
-<wire x1="-39.37" y1="46.355" x2="-34.925" y2="46.99" width="0" layer="19" extent="1-1"/>
+<wire x1="-41.595" y1="46.355" x2="-27.305" y2="65.345" width="0" layer="19" extent="1-16"/>
+<wire x1="-39.37" y1="46.355" x2="-41.595" y2="46.355" width="0" layer="19" extent="16-16"/>
+<wire x1="-34.925" y1="46.99" x2="-39.37" y2="46.355" width="0" layer="19" extent="1-1"/>
 <wire x1="-34.925" y1="31.75" x2="-34.925" y2="46.99" width="0" layer="19" extent="1-1"/>
 <wire x1="-34.925" y1="27.305" x2="-34.925" y2="31.75" width="0" layer="19" extent="1-1"/>
@@
 <wire x1="10.795" y1="48.895" x2="-10.795" y2="59.055" width="0" layer="19" extent="1-1"/>
 <wire x1="24.13" y1="48.895" x2="10.795" y2="48.895" width="0" layer="19" extent="1-1"/>
+<wire x1="38.1" y1="48.26" x2="24.13" y2="48.895" width="0" layer="19" extent="1-1"/>
 <wire x1="6.35" y1="27.305" x2="10.795" y2="48.895" width="0" layer="19" extent="1-1"/>
-<wire x1="38.1" y1="48.26" x2="24.13" y2="48.895" width="0" layer="19" extent="1-1"/>
 <wire x1="38.1" y1="15.24" x2="38.1" y2="48.26" width="0" layer="19" extent="1-1"/>
 </signal>
@@
 <contactref element="DD3" pad="3"/>
 <contactref element="DD1" pad="2"/>
+<wire x1="16.51" y1="48.895" x2="30.48" y2="45.72" width="0" layer="19" extent="1-1"/>
 <wire x1="24.13" y1="31.115" x2="30.48" y2="45.72" width="0" layer="19" extent="1-1"/>
-<wire x1="16.51" y1="48.895" x2="24.13" y2="31.115" width="0" layer="19" extent="1-1"/>
 <wire x1="-46.99" y1="41.275" x2="16.51" y2="48.895" width="0" layer="19" extent="1-1"/>
 </signal>
@@
 <wire x1="-19.05" y1="109.54" x2="25.4" y2="119.7" width="0" layer="19" extent="1-1"/>
 <wire x1="-3.175" y1="59.055" x2="-19.05" y2="109.54" width="0" layer="19" extent="1-1"/>
+<wire x1="38.1" y1="45.72" x2="-3.175" y2="59.055" width="0" layer="19" extent="1-1"/>
 <wire x1="-46.99" y1="38.735" x2="-3.175" y2="59.055" width="0" layer="19" extent="1-1"/>
-<wire x1="38.1" y1="45.72" x2="-3.175" y2="59.055" width="0" layer="19" extent="1-1"/>
 </signal>
 <signal name="CPU-A0">
@@
 <contactref element="RV1" pad="1"/>
 <contactref element="DD3" pad="1"/>
-<wire x1="-39.37" y1="43.815" x2="-12.7" y2="109.54" width="0" layer="19" extent="1-1"/>
-<wire x1="-39.37" y1="36.195" x2="-39.37" y2="43.815" width="0" layer="19" extent="1-1"/>
-<wire x1="-46.99" y1="46.355" x2="-39.37" y2="43.815" width="0" layer="19" extent="1-1"/>
+<wire x1="-46.99" y1="46.355" x2="-42.9895" y2="45.0215" width="0.4064" layer="16"/>
+<wire x1="-42.9895" y1="45.0215" x2="-39.37" y2="43.815" width="0.4064" layer="16"/>
+<wire x1="-39.37" y1="36.195" x2="-42.9895" y2="36.195" width="0.4064" layer="16"/>
+<wire x1="-42.9895" y1="36.195" x2="-42.9895" y2="45.0215" width="0.4064" layer="16"/>
+<wire x1="-42.9895" y1="45.0215" x2="-43.495" y2="46.355" width="0" layer="19" extent="16-16"/>
 </signal>
 <signal name="N$18">
