File: KeyboardTransformer.sch (EAGLE design)
At the start: 45 parts, among them IC1 74LS09N, IC2 ли6, IC6 74LS09N, IC7 74AC10N

Commit message: .
Other:
- moved on the sheet: C1, C2, C6, D3, D4, DD1C, DD1D, DD1E, DD4B, DD5C, M, R5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
